Commit message: MZ07 simulation in moveit

File: mz07/urdf/mz07.urdf (robot description, URDF)
Before this commit: robot mz07, 8 links, 7 joints
Joints:
- joint J1: limit lower=-2.97 upper=2.97 effort=100 velocity=1 -> lower=-2.97 upper=2.97 effort=100 velocity=7.85
- joint J2: axis 0 0 1 -> 0 0 -1; limit lower=-2.36 upper=1.40 effort=100 velocity=1 -> lower=-2.36 upper=1.40 effort=100 velocity=6.63
- joint J3: limit lower=-2.37 upper=4.71 effort=100 velocity=1 -> lower=-1.169 upper=3.316 effort=100 velocity=9.08
- joint J4: limit lower=-3.32 upper=3.32 effort=100 velocity=1 -> lower=-3.32 upper=3.32 effort=100 velocity=9.60
- joint J5: limit lower=-2.09 upper=2.09 effort=100 velocity=1 -> lower=-2.09 upper=2.09 effort=100 velocity=9.60
- joint J6: limit lower=-6.28 upper=6.28 effort=100 velocity=1 -> lower=-6.28 upper=6.28 effort=100 velocity=17.50
